Commit message: Successfully imported warehouse nd navigated robot

File: src/robot_description/urdf/mybot.xacro (robot description, xacro)
@@ -7,6 +7,13 @@
   <xacro:property name="wheel_separation" value="0.15"/>
   <xacro:property name="wheel_joint_offset" value="0.02"/>
-  <xacro:property name="caster_wheel_radius" value="0.02"/>
-  <xacro:property name="caster_wheel_joint_offset" value="-0.05"/>
+  <xacro:property name="caster_wheel_radius" value="${wheel_radius/2}"/>
+  <xacro:property name="caster_wheel_mass" value="0.001"/>
+  <xacro:property name="caster_wheel_joint_offset" value="-0.052"/>
+  <xacro:property name="laser_size_x" value="0.03"/>
+  <xacro:property name="laser_size_y" value="0.03"/>
+  <xacro:property name="laser_size_z" value="0.04"/>
+  <xacro:property name="laser_origin_x" value="0.065"/>
+  <xacro:property name="laser_origin_y" value="0"/>
+  <xacro:property name="laser_origin_z" value="0.035"/>
   <xacro:macro name="box_inertia" params="m w h d">
     <inertial>
@@ -103,4 +110,23 @@
    <origin xyz="${caster_wheel_joint_offset} 0 -${caster_wheel_radius+0.005}" rpy="0 0 0"/>
  </joint>
+ <link name="sensor_laser">
+   <visual>
+      <geometry>
+        <box size="${laser_size_x} ${laser_size_y} ${laser_size_z}"/>
+      </geometry>
+      <material name="blue"/>
+    </visual>
+    <collision>
+      <geometry>
+        <box size="${laser_size_x} ${laser_size_y} ${laser_size_z}"/>
+      </geometry>
+    </collision>
+    <xacro:box_inertia m="0.2" w="${laser_size_x}" h="${laser_size_y}" d="${laser_size_z}"/>
+  </link>
+  <joint name="sensor_laser_joint" type="fixed">
+    <origin xyz="${laser_origin_x} ${laser_origin_y} ${laser_origin_z}" rpy="0 0 0" />
+    <parent link="base_link"/>
+    <child link="sensor_laser" />
+  </joint>
 <xacro:include filename="$(find robot_description)/urdf/mybot_gazebo_plugins.xacro"/>
 </robot>

File: src/robot_description/urdf/mybot_gazebo_plugins.xacro (robot description, xacro)
@@ -17,3 +17,34 @@
     </plugin>
   </gazebo>
+  <gazebo reference="sensor_laser">
+    <sensor type="gpu_ray" name="head_hokuyo_sensor">
+      <pose>0 0 0 0 0 0</pose>
+      <visualize>true</visualize>
+      <update_rate>20</update_rate>
+      <ray>
+        <scan>
+          <horizontal>
+            <samples>1440</samples>
+            <resolution>1</resolution>
+            <min_angle>-3.14159</min_angle>
+            <max_angle>3.14159</max_angle>
+          </horizontal>
+        </scan>
+        <range>
+          <min>0.10</min>
+          <max>30.0</max>
+          <resolution>0.01</resolution>
+        </range>
+        <noise>
+          <type>gaussian</type>
+          <mean>0.0</mean>
+          <stddev>0.01</stddev>
+        </noise>
+      </ray>
+      <plugin name="gazebo_ros_head_hokuyo_controller" filename="libgazebo_ros_gpu_laser.so">
+        <topicName>/mybot/laser_scan/scan</topicName>
+        <frameName>sensor_laser</frameName>
+      </plugin>
+    </sensor>
+  </gazebo>
 </robot>

Commit message: 2D SLAM working

File: src/robot_description/urdf/mybot.xacro (robot description, xacro)
@@ -84,9 +84,9 @@
     <xacro:wheel prefix="right" reflect="-1"/>
     <xacro:macro name="sphere_inertia" params="m r">
-   <inertial>
-     <mass value="${m}"/>
-     <inertia ixx="${2.0*m*(r*r)/5.0}" ixy="0.0" ixz="0.0" iyy="${2.0*m*(r*r)/5.0}" iyz="0.0" izz="${2.0*m*(r*r)/5.0}"/>
-   </inertial>
- </xacro:macro>
+     <inertial>
+       <mass value="${m}"/>
+       <inertia ixx="${2.0*m*(r*r)/5.0}" ixy="0.0" ixz="0.0" iyy="${2.0*m*(r*r)/5.0}" iyz="0.0" izz="${2.0*m*(r*r)/5.0}"/>
+     </inertial>
+   </xacro:macro>
   <link name="caster_wheel">
    <visual>

File: src/robot_description/urdf/mybot_gazebo_plugins.xacro (robot description, xacro)
@@ -12,5 +12,5 @@
       <torque>20</torque>
       <commandTopic>/mybot/base_controller/cmd_vel</commandTopic>
-      <odometryTopic>/mybot/base_controller/odom</odometryTopic>
+      <odometryTopic>odom</odometryTopic>
       <odometryFrame>odom</odometryFrame>
       <robotBaseFrame>base_footprint</robotBaseFrame>
@@ -43,5 +43,5 @@
       </ray>
       <plugin name="gazebo_ros_head_hokuyo_controller" filename="libgazebo_ros_gpu_laser.so">
-        <topicName>/mybot/laser_scan/scan</topicName>
+        <topicName>scan</topicName>
         <frameName>sensor_laser</frameName>
       </plugin>
